File: Board/Eagle Files RISC-V-Brain/Brain_0.1.rv1.sch (EAGLE design)
At the start: 30 parts, among them U1 U1, Y1 Y1YSX211SL, Y2 32.768K

Commit message: Update Eagles Files add files for assembly
Parts:
- LED, PWD: value (none) -> LED
- R8: LCSC_PART C25744 -> (none)
Changed lines of the file:
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@@
 <attribute name="PRICE-1000" value="0.0005"/>
 </part>
-<part name="PWD" library="CH582M" library_urn="urn:adsk.eagle:library:36586898" deviceset="LED" device="" package3d_urn="urn:adsk.eagle:package:38116458/5">
+<part name="PWD" library="CH582M" library_urn="urn:adsk.eagle:library:36586898" deviceset="LED" device="" package3d_urn="urn:adsk.eagle:package:38116458/5" value="LED">
 <attribute name="LCSC" value="C434447"/>
 <attribute name="PRICE-1" value="0.0140"/>
@@
 <attribute name="PRICE-1000" value="0.0111"/>
 </part>
-<part name="LED" library="CH582M" library_urn="urn:adsk.eagle:library:36586898" deviceset="LED" device="" package3d_urn="urn:adsk.eagle:package:38116458/5">
+<part name="LED" library="CH582M" library_urn="urn:adsk.eagle:library:36586898" deviceset="LED" device="" package3d_urn="urn:adsk.eagle:package:38116458/5" value="LED">
 <attribute name="LCSC" value="C434447"/>
 <attribute name="PRICE-1" value="0.0140"/>
@@
 </spice>
 <attribute name="LCSC" value="C25744"/>
-<attribute name="LCSC_PART" value="C25744"/>
 <attribute name="PRICE-1" value="0.0006"/>
 <attribute name="PRICE-100" value="0.0006"/>
